File: expansionboardA.kicad_pcb (KiCad board)
At the start: 2 copper layers, 111 x 109.4 mm, 51 parts, among them J1 DEBUG, J2 USB_A_Stacked, J3 HDMI_A, J4 FAN, P1 USB_C_Plug, U1 MAX3420EECJ, U2 GPIO_U2, U3 AMS1117-3.3, U4 GPIO_U4, U5 MCP3008T-I/SL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

Commit message: Updated board
Parts:
- added RESETN1: SW_Push, 1_1825027_1:SW_1-1825027-1, B.Cu at (124.5, 48.3)
- moved C3 7.26 mm to (80.7, 86.6), turned to 0 degrees
- moved Y1 1.80 mm to (85.2, 88.8), turned to -90 degrees
- moved C4 1.37 mm to (80.7, 93.5), turned to 0 degrees
Connections:
- U4 pad 59: unconnected-(U4-Pin_59-Pad59) -> RSTN
Routing:
- net /input3v3: track 213.5 -> 184.4 mm, vias 6 -> 5
- net RSTN: track 0.00 -> 16.2 mm
- net /AL: track 82.9 -> 74.4 mm
- net Net-(U1-XO): track 8.64 -> 13.1 mm
- net Net-(U1-XI): track 8.68 -> 13.1 mm
- net /AR: track 78.2 -> 74.3 mm
- net USBGPIN3: track 44.1 -> 42.2 mm
- net USBGPIN2: track 41.3 -> 39.8 mm
- net USBGPIN1: track 44.4 -> 43.2 mm
- net USBGPIN0: track 41.5 -> 40.6 mm
- net GND: track 33.0 -> 33.1 mm, vias 27 -> 26
Other:
- board text added: "RESET"
