File: expansionboardA.kicad_sch (KiCad schematic)
At the start: 51 parts, among them J1 DEBUG, J2 USB_A_Stacked, J3 HDMI_A, J4 FAN, P1 USB_C_Plug, U1 MAX3420EECJ, U2 GPIO_U2, U3 AMS1117-3.3, U4 GPIO_U4, U5 MCP3008T-I/SL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

Commit message: Updated board
Parts:
- added RESETN1: SW_Push, SW_1-1825027-1, symbol 1-1825027-1:1-1825027-1
Connections:
- net GND: now also RESETN1.1
- net RSTN: now reaches U4.59 (Pin_59)
- net RSTN: now also RESETN1.2
Other:
- note added: "RESET"
Changed lines of the file:
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@@
+    (stroke (width 0) (type default))
+  )
+  (wire (pts (xy 173.99 153.67) (xy 176.53 153.67))
     (stroke (width 0) (type default))
   )
@@
     (stroke (width 0) (type default))
   )
+  (wire (pts (xy 245.11 151.13) (xy 246.38 151.13))
+    (stroke (width 0) (type default))
+  )
   (wire (pts (xy 389.89 45.72) (xy 387.35 45.72))
     (stroke (width 0) (type default))
@@
     (stroke (width 0) (type default))
   )
+  (wire (pts (xy 158.75 153.67) (xy 158.75 158.75))
+    (stroke (width 0) (type default))
+  )
   (wire (pts (xy 322.58 101.6) (xy 322.58 99.06))
     (stroke (width 0) (type default))
@@
   )
   (rectangle (start 274.32 67.31) (end 403.86 227.33)
+    (stroke (width 0) (type default))
+    (fill (type none))
+  )
+  (rectangle (start 151.13 144.78) (end 184.15 165.1)
     (stroke (width 0) (type default))
     (fill (type none))
@@
     (effects (font (size 1.27 1.27)) (justify left bottom))
   )
+  (text "RESET" (at 152.4 147.32 0)
+    (effects (font (size 1.27 1.27)) (justify left bottom))
+  )
   (text "3v3 Power Regulator" (at 215.9 17.78 0)
     (effects (font (size 1.27 1.27)) (justify left bottom))
@@
     )
   )
+  (global_label "GND" (shape input) (at 158.75 158.75 180) (fields_autoplaced)
+    (effects (font (size 1.27 1.27)) (justify right))
+    (property "Intersheetrefs" "${INTERSHEET_REFS}" (at 151.9737 158.75 0)
+      (effects (font (size 1.27 1.27)) (justify right) hide)
+    )
+  )
   (global_label "LED2" (shape output) (at 200.66 139.7 180) (fields_autoplaced)
     (effects (font (size 1.27 1.27)) (justify right))
@@
     )
   )
+  (global_label "RSTN" (shape input) (at 245.11 151.13 180) (fields_autoplaced)
+    (effects (font (size 1.27 1.27)) (justify right))
+    (property "Intersheetrefs" "${INTERSHEET_REFS}" (at 237.4266 151.13 0)
+      (effects (font (size 1.27 1.27)) (justify right) hide)
+    )
+  )
   (global_label "AU_SDIN" (shape input) (at 200.66 114.3 180) (fields_autoplaced)
     (effects (font (size 1.27 1.27)) (justify right))
@@
     (property "Intersheetrefs" "${INTERSHEET_REFS}" (at 189.5899 116.84 0)
       (effects (font (size 1.27 1.27)) (justify right) hide)
+    )
+  )
+  (global_label "RSTN" (shape input) (at 176.53 153.67 0) (fields_autoplaced)
+    (effects (font (size 1.27 1.27)) (justify left))
+    (property "Intersheetrefs" "${INTERSHEET_REFS}" (at 184.2134 153.67 0)
+      (effects (font (size 1.27 1.27)) (justify left) hide)
     )
   )
@@
         )
       )
+    )
+  )
+  (symbol (lib_id "1-1825027-1:1-1825027-1") (at 166.37 156.21 0) (unit 1)
+    (in_bom yes) (on_board yes) (dnp no) (fields_autoplaced)
+    (property "Reference" "RESETN1" (at 166.37 147.32 0)
+      (effects (font (size 1.27 1.27)))
+    )
+    (property "Value" "SW_Push" (at 166.37 149.86 0)
+      (effects (font (size 1.27 1.27)))
+    )
+    (property "Footprint" "SW_1-1825027-1" (at 166.37 156.21 0)
+      (effects (font (size 1.27 1.27)) (justify left bottom) hide)
+    )
+    (property "Datasheet" "~" (at 166.37 156.21 0)
+      (effects (font (size 1.27 1.27)) (justify left bottom) hide)
+    )
+    (property "PARTREV" "G4" (at 166.37 156.21 0)
+      (effects (font (size 1.27 1.27)) (justify left bottom) hide)
+    )
+    (property "STANDARD" "Manufacturer Recommednation" (at 166.37 156.21 0)
+      (effects (font (size 1.27 1.27)) (justify left bottom) hide)
+    )
+    (property "MANUFACTURER" "TE Connectivity" (at 166.37 156.21 0)
+      (effects (font (size 1.27 1.27)) (justify left bottom) hide)
+    )
+    (pin "1")
+    (pin "2")
+    (pin "S1")
+    (pin "S2")
+    (instances
+      (project "expansionboardA"
+        (path "/317f7f3e-4535-46d0-9a87-af1bea12706a"
+          (reference "RESETN1") (unit 1)
+        )
+      )
